File: PA 500mW for SX1255.kicad_pcb (KiCad board)
At the start: 2 copper layers, 67.5 x 30.8 mm, 33 parts, among them J1 RF-in, J2 RF-out, J3 5Vcc input, U2 TQP7M9106

Commit message: Add files via upload
Parts:
- removed FL1: LFCN-490, Filter:Filter_Mini-Circuits_FV1206
- removed the REF** at (158.2, 95.0)
- added REF**: OSHW-Logo2_7.3x6mm_SilkScreen, Symbol:OSHW-Logo2_7.3x6mm_SilkScreen, F.Cu at (157.0, 95.8)
- moved C12 4.00 mm to (157.2, 108.9)
- moved C18 3.64 mm to (113.4, 98.9)
- moved J3 3.50 mm to (111.8, 92.8)
- moved L5 3.50 mm to (118.5, 93.0)
- moved C17 3.25 mm to (122.5, 94.2)
- moved J1 3.00 mm to (106.5, 109.1)
- moved J2 2.53 mm to (162.8, 108.9)
- moved C11 2.00 mm to (151.5, 109.7)
- moved C10 1.00 mm to (144.0, 109.6)
- moved C6 0.56 mm to (122.2, 110.0)
- moved L4 0.51 mm to (146.2, 108.9)
- moved C13 0.25 mm to (143.0, 102.2)
- moved C14 0.25 mm to (143.0, 98.2)
- moved C15 0.25 mm to (143.0, 96.5)
- moved C16 0.25 mm to (143.8, 93.0)
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Connections:
- C12 pad 2: Net-(FL1-IN) -> Net-(FL1-OUT)
Routing:
- net Net-(C13-Pad1): track 41.8 -> 27.4 mm
- net /RF_OUT/VCC: track 10.3 -> 0.00 mm
- net Net-(J1-In): track 8.72 -> 0.00 mm
- net Net-(C5-Pad1): track 7.45 -> 0.00 mm
- net /RF_IN: track 6.94 -> 0.00 mm
- net Net-(C11-Pad2): track 5.94 -> 0.00 mm
- net Net-(FL1-OUT): track 5.70 -> 0.00 mm
- net Net-(U2-VBIAS): track 11.8 -> 6.37 mm
- net Net-(C4-Pad1): track 5.10 -> 0.00 mm
- net Net-(U2-I_REF): track 5.09 -> 0.00 mm
- net Net-(FL1-IN): track 2.48 -> 0.00 mm
- net GND: track 16.0 -> 15.3 mm, vias 38 -> 65
- added copper zone on F.Cu, net Net-(C11-Pad2)
- added copper zone on F.Cu, net Net-(C13-Pad1)
- added copper zone on F.Cu, net Net-(C4-Pad1)
- added copper zone on F.Cu, net Net-(C5-Pad1)
- added copper zone on F.Cu, net Net-(FL1-OUT)
- added copper zone on F.Cu, net Net-(J1-In)
- added copper zone on F.Cu, net Net-(U2-I_REF)
- added copper zone on F.Cu, net Net-(U2-VBIAS)
Other:
- board size 67.5 x 30.8 mm -> 61.8 x 30.8 mm
- board text added: "BIAS"
- board text added: "PA"
