File: PA 500mW for SX1255.kicad_pcb (KiCad board)
At the start: 2 copper layers, 61.8 x 30.8 mm, 32 parts, among them J1 RF-in, J2 RF-out, J3 5Vcc input, U2 TQP7M9106

Commit message: Add files via upload
Parts:
- added D1: SP0502BAHT, Package_TO_SOT_SMD:SOT-23-3, F.Cu at (106.8, 99.1)
- added H3: MountingHole, MountingHole:MountingHole_2.2mm_M2_DIN965_Pad, F.Cu at (116.0, 100.2)
- added H5: MountingHole, MountingHole:MountingHole_2.2mm_M2_DIN965_Pad, F.Cu at (116.0, 116.0)
- added R5: 10R, Resistor_SMD:R_0603_1608Metric, F.Cu at (138.8, 97.5)
- added R6: 10R, Resistor_SMD:R_0603_1608Metric, F.Cu at (130.8, 97.5)
- C16, C18: footprint Capacitor_Tantalum_SMD:CP_EIA-3528-15_AVX-H_HandSolder -> Capacitor_Tantalum_SMD:CP_EIA-3216-18_Kemet-A
- J3: value 5Vcc input -> USB_C_Receptacle_PowerOnly_6P; footprint TerminalBlock:TerminalBlock_bornier-2_P5.08mm -> Connector_USB:USB_C_Receptacle_GCT_USB4125-xx-x_6P_TopMnt_Horizontal
- R3, R4: value 280R -> 270R
- moved H1 8.59 mm to (134.8, 100.2)
- moved H2 8.53 mm to (134.8, 116.2)
- moved H4 5.64 mm to (154.0, 100.2)
- moved H6 5.51 mm to (154.0, 116.2)
- moved REF** 4.45 mm to (160.5, 93.0)
- moved C18 2.64 mm to (110.8, 99.0), turned to -90 degrees
- moved J3 2.55 mm to (109.2, 92.2)
- moved R3 2.50 mm to (138.8, 94.2)
- moved R4 2.50 mm to (130.8, 94.2)
- moved C16 0.25 mm to (143.5, 93.0)
- moved C8 0.25 mm to (139.5, 100.5)
Connections:
- C18 pad 1: +5V -> Net-(C18-Pad1)
- H1 pad 1: GND -> (no net)
- H2 pad 1: GND -> (no net)
- H4 pad 1: GND -> (no net)
- H6 pad 1: GND -> (no net)
- L5 pad 1: +5V -> Net-(C18-Pad1)
- R3 pad 2: Net-(C8-Pad1) -> Net-(R3-Pad2)
- R4 pad 2: Net-(U2-VBIAS) -> Net-(R4-Pad2)
- U2 pad 27: GND -> (no net)
- U2 pad 28: GND -> (no net)
- U2 pad 29: GND -> (no net)
- U2 pad 30: GND -> (no net)
- U2 pad 31: GND -> (no net)
- U2 pad 32: GND -> (no net)
- U2 pad 33: GND -> (no net)
- U2 pad 34: GND -> (no net)
- U2 pad 35: GND -> (no net)
- U2 pad 36: GND -> (no net)
- U2 pad 37: GND -> (no net)
- U2 pad 38: GND -> (no net)
- U2 pad 39: GND -> (no net)
- U2 pad 40: GND -> (no net)
- U2 pad 41: GND -> (no net)
- U2 pad 42: GND -> (no net)
Routing:
- net +5V: track 12.2 -> 0.00 mm
- net GND: track 15.3 -> 25.6 mm, vias 65 -> 59
- net Net-(C18-Pad1): track 0.00 -> 7.61 mm
- net Net-(C13-Pad1): track 27.4 -> 22.1 mm
- net Net-(R4-Pad2): track 0.00 -> 1.60 mm
- net Net-(R3-Pad2): track 0.00 -> 1.60 mm
- net Net-(U2-VBIAS): track 6.37 -> 5.42 mm
- net Net-(C8-Pad1): track 4.64 -> 3.89 mm
- added copper zone on F.Cu, net Net-(C18-Pad1)
