File: PA 500mW for SX1255.kicad_sch (KiCad schematic)
At the start: 33 parts, among them J1 RF-in, J2 RF-out, J3 5Vcc input, U2 TQP7M9106

Commit message: Add files via upload
Parts:
- removed J3: 5Vcc input, TerminalBlock:TerminalBlock_bornier-2_P5.08mm, symbol Connector:Screw_Terminal_01x02
- added D1: SP0502BAHT, Package_TO_SOT_SMD:SOT-23-3, symbol Power_Protection:SP0502BAHT
- added J3: USB_C_Receptacle_PowerOnly_6P, Connector_USB:USB_C_Receptacle_GCT_USB4125-xx-x_6P_TopMnt_Horizontal, symbol Connector:USB_C_Receptacle_PowerOnly_6P
- added R5, R6: 10R, Resistor_SMD:R_0603_1608Metric, symbol Device:R_Small
- C16: footprint Capacitor_Tantalum_SMD:CP_EIA-3528-15_AVX-H_HandSolder -> Capacitor_Tantalum_SMD:CP_EIA-3216-18_Kemet-A; DigiKey Part Number 478-1682-1-ND -> 478-1663-1-ND; Manufacturer Product Number TAJB226K016RNJ -> TAJA226K010RNJ
- C18: footprint Capacitor_Tantalum_SMD:CP_EIA-3528-15_AVX-H_HandSolder -> Capacitor_Tantalum_SMD:CP_EIA-3216-18_Kemet-A; DigiKey Part Number 478-1718-1-ND -> 478-8223-1-ND; Manufacturer Product Number TAJC476K016RNJ -> F931A476KAA
- R3, R4: value 280R -> 270R; DigiKey Part Number 541-280HCT-ND -> 541-5301-1-ND; Manufacturer Product Number CRCW0603280RFKEA -> CRCW0603270RFKEAC
Connections:
- net GND: now also D1.3 (A), J3.A12 (GND), J3.B12 (GND), J3.SH (SHIELD)
- net at C9.1, U2.1 (VBIAS): now also R6.2; no longer R4.2
- net at C8.1, L2.1: now also R5.2; no longer R3.2
- net +5V: no longer names the net of C18.1, L5.1
- net +5V: now also D1.1 (K), D1.2 (K), J3.A9 (VBUS), J3.B9 (VBUS)
- new net: R4.2, R6.1
- new net: R3.2, R5.1
- no-connect marks 0 -> 2
Other:
- moved on the sheet: R3, R4
